File: pi-pico.kicad_sch (KiCad schematic)
At the start: 14 parts, among them U1 RP2040

Commit message: IN progress Crysion Oscillator not yet configured
Parts:
- added C12, C13: C1u, Capacitor_SMD:C_0402_1005Metric_Pad0.74x0.62mm_HandSolder, symbol Device:C
- added C14: C100n, Capacitor_SMD:C_0402_1005Metric_Pad0.74x0.62mm_HandSolder, symbol Device:C
- added J1: USB_C_Receptacle_USB2.0_16P, Connector_USB:USB_C_Receptacle_G-Switch_GT-USB-7010ASV, symbol Connector:USB_C_Receptacle_USB2.0_16P
- added J2: Conn_01x02, Connector_PinHeader_2.54mm:PinHeader_1x02_P2.54mm_Vertical, symbol Connector_Generic:Conn_01x02
- added R3: R1M, Resistor_SMD:R_0402_1005Metric_Pad0.72x0.64mm_HandSolder, symbol Device:R
- added R4: R1k, Resistor_SMD:R_0402_1005Metric_Pad0.72x0.64mm_HandSolder, symbol Device:R
- added TP1: TestPoint_2Pole, TestPoint:TestPoint_2Pads_Pitch2.54mm_Drill0.8mm, symbol Connector:TestPoint_2Pole
- added U2: NCP1117-3.3_SOT223, Package_TO_SOT_SMD:SOT-223-3_TabPin2, symbol Regulator_Linear:NCP1117-3.3_SOT223
- added U3: W25Q128JVS, Package_SO:SOIC-8_5.23x5.23mm_P1.27mm, symbol Memory_Flash:W25Q128JVS
Connections:
- net +3V3: now also C13.1, C14.1, TP1.1, U2.2 (VO), U3.8 (VCC)
- net GND: now also C12.2, C13.2, C14.2, J1.A1 (GND), J1.A12 (GND), J1.B1 (GND), J1.B12 (GND), J2.1 (Pin_1), R3.2, U2.1 (GND), U3.4 (GND)
- net SCLK: now also U3.6 (CLK)
- net SD0: now also U3.5 (DI(IO0))
- net SD1: now also U3.2 (DO(IO1))
- net SD2: now also U3.3 (IO2)
- net SD3: now also U3.7 (IO3)
- net SS: now also R4.2, TP1.2, U3.1 (~{CS})
- net USB_D-: now also J1.A7 (D-)
- net USP_D+: now also J1.A6 (D+)
- new net: J1.S1 (SHIELD), R3.1
- new net: J2.2 (Pin_2), R4.1
- new net VBUS: C12.1, J1.A4 (VBUS), J1.A9 (VBUS), J1.B4 (VBUS), J1.B9 (VBUS), U2.3 (VI)

Commit message: PCB
Parts:
- added C15, C16: C15p, Capacitor_SMD:C_0402_1005Metric_Pad0.74x0.62mm_HandSolder, symbol Device:C
- added J3, J4: Conn_01x18, Connector_PinHeader_2.54mm:PinHeader_1x18_P2.54mm_Vertical, symbol Connector_Generic:Conn_01x18
- added R5: R1k, Resistor_SMD:R_0402_1005Metric_Pad0.72x0.64mm_HandSolder, symbol Device:R
- added Y1: Crystal_GND24, Crystal:Crystal_SMD_3225-4Pin_3.2x2.5mm, symbol Device:Crystal_GND24
- TP1: footprint TestPoint:TestPoint_2Pads_Pitch2.54mm_Drill0.8mm -> Resistor_SMD:R_0201_0603Metric
Connections:
- net +3V3: now also J3.1 (Pin_1)
- net ADC0: now also J4.15 (Pin_15)
- net ADC1: now also J4.16 (Pin_16)
- net ADC2: now also J4.17 (Pin_17)
- net ADC3: now also J4.18 (Pin_18)
- net GND: now also C15.1, C16.1, J3.18 (Pin_18), J4.1 (Pin_1), Y1.2, Y1.4
- net GPIO0: now also J3.2 (Pin_2)
- net GPIO1: now also J3.3 (Pin_3)
- net GPIO10: now also J3.12 (Pin_12)
- net GPIO11: now also J3.13 (Pin_13)
- net GPIO12: now also J3.14 (Pin_14)
- net GPIO13: now also J3.15 (Pin_15)
- net GPIO14: now also J3.16 (Pin_16)
- net GPIO15: now also J3.17 (Pin_17)
- net GPIO16: now also J4.5 (Pin_5)
- net GPIO17: now also J4.6 (Pin_6)
- net GPIO18: now also J4.7 (Pin_7)
- net GPIO19: now also J4.8 (Pin_8)
- net GPIO2: now also J3.4 (Pin_4)
- net GPIO20: now also J4.9 (Pin_9)
- net GPIO21: now also J4.10 (Pin_10)
- net GPIO22: now also J4.11 (Pin_11)
- net GPIO23: now also J4.12 (Pin_12)
- net GPIO24: now also J4.13 (Pin_13)
- net GPIO25: now also J4.14 (Pin_14)
- net GPIO3: now also J3.5 (Pin_5)
- net GPIO4: now also J3.6 (Pin_6)
- net GPIO5: now also J3.7 (Pin_7)
- net GPIO6: now also J3.8 (Pin_8)
- net GPIO7: now also J3.9 (Pin_9)
- net GPIO8: now also J3.10 (Pin_10)
- net GPIO9: now also J3.11 (Pin_11)
- net RUN: now also J4.4 (Pin_4)
- net SWCLK: now also J4.2 (Pin_2)
- net SWD: now also J4.3 (Pin_3)
- net XIN: now also C15.2, Y1.1
- net XOUT: now also R5.2
- new net: C16.2, R5.1, Y1.3
Other:
- moved on the sheet: C14, J2, R4, TP1, U3
