File: pi-pico.kicad_pcb (KiCad board)
At the start: 2 copper layers, 22 parts, among them J1 USB_C_Receptacle_USB2.0_16P, U1 RP2040, U2 NCP1117-3.3_SOT223, U3 W25Q128JVS

Commit message: PCB
Parts:
- added C15: C15p, Capacitor_SMD:C_0402_1005Metric_Pad0.74x0.62mm_HandSolder, F.Cu at (129.8, 87.4)
- added C16: C15p, Capacitor_SMD:C_0402_1005Metric_Pad0.74x0.62mm_HandSolder, F.Cu at (129.8, 89.3)
- added J2: Conn_01x02, Connector_PinHeader_2.54mm:PinHeader_1x02_P2.54mm_Vertical, F.Cu at (111.0, 64.2)
- added J3: Conn_01x18, Connector_PinHeader_2.54mm:PinHeader_1x18_P2.54mm_Vertical, F.Cu at (149.2, 51.9)
- added J4: Conn_01x18, Connector_PinHeader_2.54mm:PinHeader_1x18_P2.54mm_Vertical, F.Cu at (106.0, 69.1)
- added R4: R1k, Resistor_SMD:R_0402_1005Metric_Pad0.72x0.64mm_HandSolder, F.Cu at (118.0, 64.7)
- added R5: R1k, Resistor_SMD:R_0402_1005Metric_Pad0.72x0.64mm_HandSolder, F.Cu at (129.8, 85.4)
- added Y1: Crystal_GND24, Crystal:Crystal_SMD_3225-4Pin_3.2x2.5mm, F.Cu at (122.0, 87.6)
- TP1: footprint Connector_PinHeader_1.00mm:PinHeader_2x01_P1.00mm_Vertical_SMD -> Resistor_SMD:R_0201_0603Metric
- moved U1 61.8 mm to (132.5, 60.5), turned to -90 degrees
- moved U3 45.1 mm to (142.8, 60.5), turned to -90 degrees
- moved J1 42.5 mm to (104.2, 60.5), turned to -90 degrees
- moved U2 36.5 mm to (113.5, 58.8)
Other:
- board outline added: 51 x 21 mm

Commit message: COMPLETED
Parts:
- moved R1 70.4 mm to (139.2, 60.6), turned to -90 degrees
- moved R2 70.2 mm to (139.3, 63.1), turned to -90 degrees
- moved C6 61.9 mm to (121.2, 55.3), turned to -90 degrees
- moved C11 61.3 mm to (138.4, 65.8)
- moved C5 59.6 mm to (120.1, 55.3), turned to -90 degrees
- moved C10 59.1 mm to (125.5, 55.3), turned to -90 degrees
- moved C4 57.4 mm to (119.0, 55.3), turned to -90 degrees
- moved C9 56.9 mm to (124.4, 55.3), turned to -90 degrees
- moved C3 55.9 mm to (127.0, 61.1), turned to 180 degrees
- moved C8 54.7 mm to (123.3, 55.3), turned to -90 degrees
- moved C7 52.4 mm to (122.2, 55.3), turned to -90 degrees
- moved C13 49.2 mm to (116.7, 54.4), turned to 180 degrees
- moved C2 48.7 mm to (121.8, 64.2), turned to -90 degrees
- moved C1 48.0 mm to (123.0, 64.2), turned to -90 degrees
- moved TP1 45.5 mm to (142.3, 65.5), turned to 180 degrees
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Routing:
- net +3V3: track 0.00 -> 73.3 mm, vias 0 -> 1
- net /SS: track 0.00 -> 58.0 mm, vias 0 -> 3
- net /USB_D-: track 0.00 -> 37.8 mm, vias 0 -> 2
- net /USP_D+: track 0.00 -> 36.7 mm, vias 0 -> 2
- net Net-(J1-SHIELD): track 0.00 -> 32.0 mm
- net /SWCLK: track 0.00 -> 25.6 mm, vias 0 -> 1
- net GND: track 0.00 -> 24.8 mm, vias 0 -> 6
- net /GPIO15: track 0.00 -> 23.7 mm, vias 0 -> 1
- net Net-(U1-IOVDD-Pad1): track 0.00 -> 22.4 mm
- net /GPIO14: track 0.00 -> 21.4 mm, vias 0 -> 1
- net /SWD: track 0.00 -> 21.1 mm, vias 0 -> 1
- net /RUN: track 0.00 -> 19.3 mm, vias 0 -> 1
- net /GPIO13: track 0.00 -> 18.2 mm, vias 0 -> 1
- net /GPIO16: track 0.00 -> 17.8 mm, vias 0 -> 1
- net /ADC3: track 0.00 -> 17.0 mm, vias 0 -> 1
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- added copper zone on B.Cu, net GND
- added copper zone on F.Cu, net GND
